File: Hardware/PCB_controller/untitled.kicad_sch (KiCad schematic)
At the start: 4 parts, among them SW3 SW_SPST

Commit message: finished controller pcb
Connections:
- net +3V3 renamed +3.3V
Changed lines of the file:
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@@
+	(wire
+		(pts
+			(xy 127 100.33) (xy 127 106.68)
+		)
+		(stroke
+			(width 0)
+			(type default)
+		)
+	)
 	(wire
 		(pts
@@
 	(wire
 		(pts
+			(xy 127 73.66) (xy 127 74.93)
+		)
+		(stroke
+			(width 0)
+			(type default)
+		)
+	)
+	(wire
+		(pts
 			(xy 111.76 85.09) (xy 111.76 88.9)
 		)
@@
 	(wire
 		(pts
-			(xy 127 72.39) (xy 127 74.93)
-		)
-		(stroke
-			(width 0)
-			(type default)
-		)
-	)
-	(wire
-		(pts
 			(xy 111.76 85.09) (xy 115.57 85.09)
-		)
-		(stroke
-			(width 0)
-			(type default)
-		)
-	)
-	(wire
-		(pts
-			(xy 127 100.33) (xy 127 101.6)
 		)
 		(stroke
@@
 				)
 				(path "/40ae7190-86d3-4081-9749-de8a7d59eef1/7b6fd0d2-8436-48ac-895c-e7c6f98813bc"
-					(reference "C?")
+					(reference "C19")
 					(unit 1)
 				)
@@
 	)
 	(symbol
-		(lib_id "power:+3V3")
-		(at 127 72.39 0)
+		(lib_id "power:+3.3V")
+		(at 127 73.66 0)
 		(unit 1)
 		(exclude_from_sim no)
@@
 		(dnp no)
 		(fields_autoplaced yes)
-		(property "Reference" "#PWR010"
-			(at 127 76.2 0)
-			(effects
-				(font
-					(size 1.27 1.27)
-				)
-				(hide yes)
-			)
-		)
-		(property "Value" "+3V3"
-			(at 127 67.31 0)
+		(property "Reference" "#PWR024"
+			(at 127 77.47 0)
+			(effects
+				(font
+					(size 1.27 1.27)
+				)
+				(hide yes)
+			)
+		)
+		(property "Value" "+3.3V"
+			(at 127 68.58 0)
 			(effects
 				(font
@@
 		)
 		(property "Footprint" ""
-			(at 127 72.39 0)
+			(at 127 73.66 0)
 			(effects
 				(font
@@
 		)
 		(property "Datasheet" ""
-			(at 127 72.39 0)
-			(effects
-				(font
-					(size 1.27 1.27)
-				)
-				(hide yes)
-			)
-		)
-		(property "Description" "Power symbol creates a global label with name \"+3V3\""
-			(at 127 72.39 0)
+			(at 127 73.66 0)
+			(effects
+				(font
+					(size 1.27 1.27)
+				)
+				(hide yes)
+			)
+		)
+		(property "Description" "Power symbol creates a global label with name \"+3.3V\""
+			(at 127 73.66 0)
 			(effects
 				(font
@@
 		)
 		(instances
-			(project "PCB_controller"
+			(project ""
 				(path "/40ae7190-86d3-4081-9749-de8a7d59eef1/063fb2c4-95db-4bbb-938e-55d002ff434b"
+					(reference "#PWR012")
+					(unit 1)
+				)
+				(path "/40ae7190-86d3-4081-9749-de8a7d59eef1/355fd775-a379-4268-8c19-30560ae40d6c"
 					(reference "#PWR010")
 					(unit 1)
 				)
-				(path "/40ae7190-86d3-4081-9749-de8a7d59eef1/355fd775-a379-4268-8c19-30560ae40d6c"
+				(path "/40ae7190-86d3-4081-9749-de8a7d59eef1/43847174-ce9c-45b8-baf2-c7a56a10ed95"
+					(reference "#PWR026")
+					(unit 1)
+				)
+				(path "/40ae7190-86d3-4081-9749-de8a7d59eef1/4cc0bab6-15a5-4281-8501-745c5f6795d1"
+					(reference "#PWR040")
+					(unit 1)
+				)
+				(path "/40ae7190-86d3-4081-9749-de8a7d59eef1/7b6fd0d2-8436-48ac-895c-e7c6f98813bc"
 					(reference "#PWR08")
 					(unit 1)
 				)
-				(path "/40ae7190-86d3-4081-9749-de8a7d59eef1/43847174-ce9c-45b8-baf2-c7a56a10ed95"
+				(path "/40ae7190-86d3-4081-9749-de8a7d59eef1/9fe8bb3c-e039-497c-86a5-e3b1a07d09b7"
+					(reference "#PWR014")
+					(unit 1)
+				)
+				(path "/40ae7190-86d3-4081-9749-de8a7d59eef1/ac02917d-6847-4a4a-b14d-f12979707db3"
+					(reference "#PWR016")
+					(unit 1)
+				)
+				(path "/40ae7190-86d3-4081-9749-de8a7d59eef1/d61021ac-9546-4c06-a574-6490fa5d0afb"
+					(reference "#PWR022")
+					(unit 1)
+				)
+				(path "/40ae7190-86d3-4081-9749-de8a7d59eef1/e9dd2b6a-fb6c-4ba3-b85a-e90ed214800d"
 					(reference "#PWR024")
 					(unit 1)
 				)
-				(path "/40ae7190-86d3-4081-9749-de8a7d59eef1/4cc0bab6-15a5-4281-8501-745c5f6795d1"
-					(reference "#PWR026")
-					(unit 1)
-				)
-				(path "/40ae7190-86d3-4081-9749-de8a7d59eef1/7b6fd0d2-8436-48ac-895c-e7c6f98813bc"
-					(reference "#PWR?")
-					(unit 1)
-				)
-				(path "/40ae7190-86d3-4081-9749-de8a7d59eef1/9fe8bb3c-e039-497c-86a5-e3b1a07d09b7"
-					(reference "#PWR012")
-					(unit 1)
-				)
-				(path "/40ae7190-86d3-4081-9749-de8a7d59eef1/ac02917d-6847-4a4a-b14d-f12979707db3"
-					(reference "#PWR014")
-					(unit 1)
-				)
-				(path "/40ae7190-86d3-4081-9749-de8a7d59eef1/d61021ac-9546-4c06-a574-6490fa5d0afb"
+				(path "/40ae7190-86d3-4081-9749-de8a7d59eef1/ee940f34-aadb-4e1c-b5aa-aa0b827bc509"
+					(reference "#PWR018")
+					(unit 1)
+				)
+				(path "/40ae7190-86d3-4081-9749-de8a7d59eef1/fad6e345-bfb9-4f2f-846c-c423c0eba2a7"
 					(reference "#PWR020")
-					(unit 1)
-				)
-				(path "/40ae7190-86d3-4081-9749-de8a7d59eef1/e9dd2b6a-fb6c-4ba3-b85a-e90ed214800d"
-					(reference "#PWR022")
-					(unit 1)
-				)
-				(path "/40ae7190-86d3-4081-9749-de8a7d59eef1/ee940f34-aadb-4e1c-b5aa-aa0b827bc509"
-					(reference "#PWR016")
-					(unit 1)
-				)
-				(path "/40ae7190-86d3-4081-9749-de8a7d59eef1/fad6e345-bfb9-4f2f-846c-c423c0eba2a7"
-					(reference "#PWR018")
 					(unit 1)
 				)
@@
 	(symbol
 		(lib_id "power:GND")
-		(at 127 101.6 0)
+		(at 127 106.68 0)
 		(unit 1)
 		(exclude_from_sim no)
@@
 		(fields_autoplaced yes)
 		(property "Reference" "#PWR011"
-			(at 127 107.95 0)
+			(at 127 113.03 0)
 			(effects
 				(font
@@
 		)
 		(property "Value" "GND"
+			(at 127 111.76 0)
+			(effects
+				(font
+					(size 1.27 1.27)
+				)
+			)
+		)
+		(property "Footprint" ""
 			(at 127 106.68 0)
 			(effects
@@
 					(size 1.27 1.27)
 				)
-			)
-		)
-		(property "Footprint" ""
-			(at 127 101.6 0)
-			(effects
-				(font
-					(size 1.27 1.27)
-				)
 				(hide yes)
 			)
 		)
 		(property "Datasheet" ""
-			(at 127 101.6 0)
+			(at 127 106.68 0)
 			(effects
 				(font
@@
 		)
 		(property "Description" "Power symbol creates a global label with name \"GND\" , ground"
-			(at 127 101.6 0)
+			(at 127 106.68 0)
 			(effects
 				(font
@@
 				)
 				(path "/40ae7190-86d3-4081-9749-de8a7d59eef1/7b6fd0d2-8436-48ac-895c-e7c6f98813bc"
-					(reference "#PWR?")
+					(reference "#PWR041")
 					(unit 1)
 				)
@@
 				)
 				(path "/40ae7190-86d3-4081-9749-de8a7d59eef1/7b6fd0d2-8436-48ac-895c-e7c6f98813bc"
-					(reference "R?")
+					(reference "R1")
 					(unit 1)
 				)
@@
 				)
 				(path "/40ae7190-86d3-4081-9749-de8a7d59eef1/7b6fd0d2-8436-48ac-895c-e7c6f98813bc"
-					(reference "SW?")
-					(unit 1)
-				)
+					(reference "SW1")
+					(unit 1)
+				)

Commit message: started controller PCB
Parts:
- C9: value C -> 10n; footprint (none) -> Capacitor_SMD:C_0402_1005Metric_Pad0.74x0.62mm_HandSolder
- R5, R6: value R -> 10k; footprint (none) -> Resistor_SMD:R_0402_1005Metric_Pad0.72x0.64mm_HandSolder
- SW3: footprint (none) -> maker:botan
Changed lines of the file:
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@@
 			)
 		)
-		(property "Value" "C"
+		(property "Value" "10n"
 			(at 115.57 93.9799 0)
 			(effects
@@
 			)
 		)
-		(property "Footprint" ""
+		(property "Footprint" "Capacitor_SMD:C_0402_1005Metric_Pad0.74x0.62mm_HandSolder"
 			(at 112.7252 96.52 0)
 			(effects
@@
 		(dnp no)
 		(fields_autoplaced yes)
-		(property "Reference" "#PWR024"
+		(property "Reference" "#PWR012"
 			(at 127 77.47 0)
 			(effects
@@
 			)
 		)
-		(property "Value" "R"
+		(property "Value" "10k"
 			(at 119.38 81.28 90)
 			(effects
@@
 			)
 		)
-		(property "Footprint" ""
+		(property "Footprint" "Resistor_SMD:R_0402_1005Metric_Pad0.72x0.64mm_HandSolder"
 			(at 119.38 86.868 90)
 			(effects
@@
 			)
 		)
-		(property "Value" "R"
+		(property "Value" "10k"
 			(at 129.54 80.0099 0)
 			(effects
@@
 			)
 		)
-		(property "Footprint" ""
+		(property "Footprint" "Resistor_SMD:R_0402_1005Metric_Pad0.72x0.64mm_HandSolder"
 			(at 125.222 78.74 90)
 			(effects
@@
 			)
 		)
-		(property "Footprint" ""
+		(property "Footprint" "maker:botan"
 			(at 127 92.71 0)
 			(effects

Commit message: applied changes
Parts:
- renumbered C9 to C19, R6 to R1, R5 to R2, SW3 to SW1
Changed lines of the file:
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@@
 (kicad_sch
-	(version 20231120)
+	(version 20250114)
 	(generator "eeschema")
-	(generator_version "8.0")
+	(generator_version "9.0")
 	(paper "A4")
 	(junction
@@
 		(dnp no)
 		(fields_autoplaced yes)
-		(property "Reference" "C9"
+		(property "Reference" "C19"
 			(at 115.57 91.4399 0)
 			(effects
@@
 		(dnp no)
 		(fields_autoplaced yes)
-		(property "Reference" "#PWR012"
+		(property "Reference" "#PWR08"
 			(at 127 77.47 0)
 			(effects
@@
 		(dnp no)
 		(fields_autoplaced yes)
-		(property "Reference" "R5"
+		(property "Reference" "R2"
 			(at 119.38 78.74 90)
 			(effects
@@
 		(dnp no)
 		(fields_autoplaced yes)
-		(property "Reference" "#PWR011"
+		(property "Reference" "#PWR041"
 			(at 127 113.03 0)
 			(effects
@@
 		(dnp no)
 		(fields_autoplaced yes)
-		(property "Reference" "R6"
+		(property "Reference" "R1"
 			(at 129.54 77.4699 0)
 			(effects
@@
 		(dnp no)
 		(fields_autoplaced yes)
-		(property "Reference" "SW3"
+		(property "Reference" "SW1"
 			(at 129.54 91.4399 90)
 			(effects
