File: Hardware/PCB_controller/PCB_controller.kicad_pcb (KiCad board)
At the start: 4 copper layers, 46.5 x 59 mm, 72 parts, among them J1 Conn_01x02, J2 Conn_01x06, J3 Conn_01x04, J4 Conn_ST_STDC14, SW1 SW_SPST, SW10 SW_SPST, SW11 SW_SPST, SW2 SW_SPST, SW3 SW_SPST, SW4 SW_SPST, SW5 SW_SPST, SW6 SW_SPST, SW7 SW_SPST, SW8 SW_SPST, SW9 SW_SPST, U1 STM32G431KBTx, U2 AZ1117-3.3

Commit message: finished controller PCB
Parts:
- moved H4 82.7 mm to (162.0, 130.0)
- moved J2 80.5 mm to (146.2, 131.0), turned to 180 degrees
- moved R22 73.1 mm to (136.3, 118.5), turned to 90 degrees
- moved SW11 72.1 mm to (130.8, 116.3), turned to 180 degrees
- moved R21 68.7 mm to (136.3, 116.2), turned to -90 degrees
- moved C17 64.4 mm to (136.3, 114.0), turned to 90 degrees
- moved C19 58.5 mm to (152.8, 109.8), turned to -90 degrees
- moved D1 55.7 mm to (132.1, 123.5)
- moved D2 55.7 mm to (132.1, 121.9)
- moved R25 55.7 mm to (134.7, 121.9)
- moved R26 55.7 mm to (134.7, 123.5)
- moved R2 54.3 mm to (152.8, 107.6), turned to 90 degrees
- moved SW1 51.1 mm to (158.3, 107.5), turned to 0 degrees
- moved R1 50.2 mm to (152.8, 105.3), turned to -90 degrees
- moved SW10 46.7 mm to (130.8, 95.5), turned to 180 degrees
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Routing:
- net GND: track 0.00 -> 80.2 mm, vias 0 -> 49
- net BTN_8: track 0.00 -> 50.4 mm, vias 0 -> 2
- net BTN_4: track 0.00 -> 37.3 mm, vias 0 -> 2
- net +3.3V: track 0.00 -> 36.8 mm, vias 0 -> 19
- net BTN_7: track 0.00 -> 33.9 mm, vias 0 -> 2
- net I2C1_SCL: track 0.00 -> 33.3 mm, vias 0 -> 2
- net BTN_6: track 0.00 -> 31.7 mm
- net I2C1_SDA: track 0.00 -> 29.5 mm, vias 0 -> 2
- net BTN_3: track 0.00 -> 27.0 mm
- net UART2_HC05_RX: track 0.00 -> 25.8 mm
- net UART2_HC05_TX: track 0.00 -> 24.5 mm, vias 0 -> 2
- net BTN_9: track 0.00 -> 22.7 mm
- net BTN_5: track 0.00 -> 20.4 mm
- net UART1_DEBUG_RX: track 0.00 -> 19.7 mm, vias 0 -> 2
- net LED1: track 0.00 -> 19.1 mm, vias 0 -> 2
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- added copper zone on In1.Cu, net +3.3V
- added copper zone on In1.Cu, net +5V
- added copper zone on B.Cu, net GND
- added copper zone on F.Cu, net GND
- added copper zone on In2.Cu, net GND
Other:
- board size 46.5 x 59 mm -> 44.1 x 80 mm

Commit message: applied changes
Parts:
- added C20: 1u, Capacitor_SMD:C_0603_1608Metric, F.Cu at (159.3, 115.8)
- C5: value 10n -> 1u; footprint Capacitor_SMD:C_0402_1005Metric_Pad0.74x0.62mm_HandSolder -> Capacitor_SMD:C_0603_1608Metric
- C6: value 1u -> 100n; footprint Capacitor_SMD:C_0603_1608Metric -> Capacitor_SMD:C_0402_1005Metric_Pad0.74x0.62mm_HandSolder
- R23, R24: value 1k -> 10k
- R25: value 1k6 -> 3k3
- R26: value 820 -> 1k6
- R27, R28: value 82 -> 700
- moved C5 24.7 mm to (142.5, 127.5), turned to 180 degrees
- moved C6 1.21 mm to (148.8, 103.6)
Connections:
- C5 pad 1: +3.3V -> +5V
Routing:
- net GND: track 80.2 -> 88.4 mm, vias 49 -> 51
- net +5V: track 5.50 -> 13.0 mm
- net +3.3V: track 36.8 -> 35.5 mm

Commit message: generated gerbers and drill files
Routing:
- net GND: vias 51 -> 82
