File: Hardware/PCB_main_unit/PCB_main_unit.kicad_pcb (KiCad board)
At the start: 4 copper layers, 60 x 60 mm, 48 parts, among them J1 Conn_01x03, J10 Conn_01x03, J11 Conn_01x03, J12 Conn_01x04, J13 Conn_01x07, J14 Conn_ST_STDC14, J15 Conn_01x03, J16 Conn_01x02, J2 Conn_01x03, J3 Conn_01x03, J4 Conn_01x03, J5 Conn_01x03, J6 Conn_01x03, J7 Conn_01x03, J8 Conn_01x03, J9 Conn_01x06, SW1 SW_SPDT, U2 STM32G474RETx, U3 AZ1117-3.3

Commit message: .
Parts:
- SW1: footprint mylib:472123010111 -> maker:power_switch
- moved J11 59.6 mm to (129.2, 108.5), turned to 90 degrees
- moved J13 52.8 mm to (173.5, 96.0), turned to -90 degrees
- moved J15 34.6 mm to (134.0, 93.0)
- moved J7 34.6 mm to (134.0, 86.5)
- moved J8 34.0 mm to (122.0, 95.0)
- moved J6 34.0 mm to (122.0, 88.5)
- moved J3 30.0 mm to (160.5, 88.0)
- moved J1 30.0 mm to (160.5, 81.5)
- moved J12 23.5 mm to (166.5, 100.5), turned to -90 degrees
- moved J5 22.0 mm to (134.0, 80.5)
- moved D4 14.2 mm to (156.3, 94.3)
- moved D6 14.2 mm to (156.3, 97.5)
- moved R4 14.2 mm to (153.6, 94.3)
- moved R6 14.2 mm to (153.6, 97.5)
- moved D5 14.2 mm to (156.3, 95.9)
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Connections:
- J13 pad 1: +3.3V -> +5V
Routing:
- added copper zone on In1.Cu, net +12V
- added copper zone on In1.Cu, net +3.3V
- added copper zone on In1.Cu, net +5V
- added copper zone on In1.Cu, net Net-(J16-Pin_2)
Other:
- board text added: "12V"
- board text added: "3V3"
- board text added: "5V"
- board text added: "DOORS"
- board text added: "FOOD"
- board text added: "HC05"
- board text added: "LIGHTS"
- board text added: "MP3"
- board text added: "XL430"

Commit message: j'ai rien a dire
Parts:
- turned C12 to 180 degrees
- turned C7 to -90 degrees
Routing:
- net +3.3V: track 0.00 -> 33.6 mm, vias 0 -> 3
- net +5V: track 0.00 -> 6.44 mm, vias 0 -> 2
- net +12V: track 0.00 -> 1.97 mm, vias 0 -> 1

Commit message: finished main unit PCB
Parts:
- moved J2 12.0 mm to (160.5, 81.5)
- moved J3 12.0 mm to (148.5, 88.0)
- moved J1 6.50 mm to (160.5, 88.0)
- moved J4 6.50 mm to (148.5, 81.5)
- moved J6 6.50 mm to (122.0, 95.0)
- moved J8 6.50 mm to (122.0, 88.5)
- moved D4 3.20 mm to (156.3, 97.5)
- moved D6 3.20 mm to (156.3, 94.3)
- moved R4 3.20 mm to (153.6, 97.5)
- moved R6 3.20 mm to (153.6, 94.3)
- moved C12 0.36 mm to (137.2, 110.8), turned to 0 degrees
- moved C6 0.36 mm to (137.2, 109.8), turned to 180 degrees
- moved C10 0.36 mm to (139.5, 109.8), turned to 180 degrees
- moved C11 0.36 mm to (139.5, 110.8), turned to 180 degrees
Routing:
- net SPI_CS: track 0.00 -> 38.3 mm, vias 0 -> 1
- net SPI_RST: track 0.00 -> 37.5 mm, vias 0 -> 1
- net SPI_DC: track 0.00 -> 36.4 mm, vias 0 -> 1
- net SPI1_SCK: track 0.00 -> 35.0 mm, vias 0 -> 1
- net UART1_DEBUG_RX: track 0.00 -> 33.8 mm, vias 0 -> 2
- net TIM2_CH3_LIGHT2: track 0.00 -> 33.1 mm, vias 0 -> 2
- net SPI1_MOSI: track 0.00 -> 32.8 mm, vias 0 -> 1
- net TIM1_CH2_DOOR2: track 0.00 -> 30.9 mm
- net UART1_DEBUG_TX: track 0.00 -> 30.2 mm, vias 0 -> 2
- net NRST: track 0.00 -> 30.0 mm, vias 0 -> 2
- net TIM1_CH1_DOOR1: track 0.00 -> 27.6 mm
- net USART2_HD_XL430: track 0.00 -> 26.7 mm, vias 0 -> 1
- net TIM2_CH2_LIGHT1: track 0.00 -> 26.3 mm
- net UART3_TX_HC05: track 0.00 -> 26.3 mm, vias 0 -> 2
- net TIM3_CH1_LIGHT4: track 0.00 -> 25.8 mm
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Other:
- board text added: "D2"

Commit message: finished main unit PCB
Parts:
- turned C7 to 90 degrees
Routing:
- net GND: track 15.8 -> 32.4 mm, vias 4 -> 57
- net +3.3V: track 46.0 -> 44.8 mm, vias 10 -> 11

Commit message: started controller PCB
Parts:
- added L1: 39n, Inductor_SMD:L_0805_2012Metric, F.Cu at (138.9, 109.4)
- C12, C3, C6: footprint Capacitor_SMD:C_0402_1005Metric_Pad0.74x0.62mm_HandSolder -> Capacitor_SMD:C_0603_1608Metric
- moved C6 2.07 mm to (136.8, 107.7)
- moved C10 1.85 mm to (139.5, 107.9)
- moved C7 1.02 mm to (140.8, 113.4), turned to 180 degrees
- moved C12 0.38 mm to (136.8, 111.0)
- moved C3 0.31 mm to (143.9, 100.2)
Routing:
- net UART3_TX_HC05: track 26.3 -> 21.0 mm, vias 2 -> 0
- net +3.3V: track 44.8 -> 48.4 mm, vias 11 -> 12
- net GND: track 32.4 -> 34.4 mm, vias 57 -> 59

Commit message: minor changes
Parts:
- moved L1 4.59 mm to (134.4, 110.3), turned to -90 degrees
- moved C10 2.00 mm to (139.5, 109.9)
- moved C6 1.80 mm to (136.8, 109.5)
Routing:
- net +3.3V: track 48.4 -> 45.4 mm
- net GND: vias 59 -> 60

Commit message: applied changes
Parts:
- removed J15, J6, J7, J8: Conn_01x03, Connector_JST:JST_EH_B3B-EH-A_1x03_P2.50mm_Vertical
- removed L1: 39n, Inductor_SMD:L_0805_2012Metric
- added C13: 1u, Capacitor_SMD:C_0603_1608Metric, F.Cu at (125.9, 92.1)
- added C14: 1u, Capacitor_SMD:C_0603_1608Metric, F.Cu at (132.7, 107.2)
- added C15: 1u, Capacitor_SMD:C_0603_1608Metric, F.Cu at (132.7, 120.4)
- added C16: 1u, Capacitor_SMD:C_0603_1608Metric, F.Cu at (125.5, 115.6)
- added C17: 1u, Capacitor_SMD:C_0603_1608Metric, F.Cu at (163.0, 107.5)
- added C18: 1u, Capacitor_SMD:C_0603_1608Metric, F.Cu at (170.0, 97.1)
- added C19: 1u, Capacitor_SMD:C_0603_1608Metric, F.Cu at (136.7, 98.5)
- added C20: 1u, Capacitor_SMD:C_0603_1608Metric, F.Cu at (148.6, 90.7)
- added C21: 1u, Capacitor_SMD:C_0603_1608Metric, F.Cu at (136.0, 90.7)
- added C22: 1u, Capacitor_SMD:C_0603_1608Metric, F.Cu at (160.9, 90.7)
- C11: value 10n -> 100n
- C12: value 1u -> 100n; footprint Capacitor_SMD:C_0603_1608Metric -> Capacitor_SMD:C_0402_1005Metric_Pad0.74x0.62mm_HandSolder
- R1: value 5k1 -> 10k
- R2: value 1k6 -> 3k3
- R3: value 820 -> 1k6
- R4, R5, R6: value 82 -> 700
- moved J4 18.4 mm to (136.0, 95.0)
- moved J5 18.0 mm to (123.3, 95.0)
- moved C11 16.5 mm to (153.4, 102.1), turned to 0 degrees
- moved J2 13.6 mm to (148.2, 87.2)
- moved J3 12.5 mm to (136.0, 87.2)
- moved H1 4.50 mm to (173.0, 86.5)
- moved H4 4.50 mm to (123.0, 86.5)
- moved C12 2.65 mm to (139.5, 111.0), turned to 180 degrees
- moved J1 0.80 mm to (160.5, 87.2)
Connections:
- J11 pad 3: TIM2_CH1_FOOD -> TIM3_CH1_FOOD
- U2 pad 12: TIM2_CH1_FOOD -> unconnected-(U2-PA0-Pad12)
- U2 pad 17: TIM2_CH4_LIGHT3 -> unconnected-(U2-PA3-Pad17)
- U2 pad 18: TIM3_CH2_LIGHT5 -> unconnected-(U2-PA4-Pad18)
- U2 pad 20: TIM3_CH1_LIGHT4 -> TIM3_CH1_FOOD
- U2 pad 43: TIM2_CH3_LIGHT2 -> unconnected-(U2-PA9-Pad43)
Routing:
- net GND: track 34.4 -> 83.4 mm, vias 60 -> 68
- net +5V: track 7.03 -> 41.7 mm
- net TIM2_CH3_LIGHT2: track 33.1 -> 0.00 mm, vias 2 -> 0
- net TIM3_CH1_LIGHT4: track 25.8 -> 0.00 mm
- net TIM2_CH4_LIGHT3: track 20.8 -> 0.00 mm
- net TIM2_CH1_FOOD: track 19.1 -> 0.00 mm, vias 1 -> 0
- net TIM3_CH2_LIGHT5: track 15.3 -> 0.00 mm
- net TIM1_CH4_GARAGE: track 25.7 -> 11.2 mm
- net TIM3_CH1_FOOD: track 0.00 -> 14.2 mm
- net TIM1_CH2_DOOR2: track 30.9 -> 18.2 mm
- net +12V: track 1.97 -> 5.85 mm
- net +3.3V: track 45.4 -> 43.4 mm, vias 12 -> 11
- net TIM1_CH1_DOOR1: track 27.6 -> 29.2 mm
- net SPI1_SCK: track 35.0 -> 33.4 mm
- net TIM2_CH2_LIGHT1: track 26.3 -> 25.1 mm, vias 0 -> 1
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Other:
- board size 60 x 60 mm -> 60 x 55.5 mm
