File: Hardware/PCB_main_unit/PCB_main_unit.kicad_pcb (KiCad board)
At the start: 4 copper layers, 60 x 55.5 mm, 54 parts, among them J1 Conn_01x03, J10 Conn_01x03, J11 Conn_01x03, J12 Conn_01x04, J13 Conn_01x07, J14 Conn_ST_STDC14, J16 Conn_01x02, J2 Conn_01x03, J3 Conn_01x03, J4 Conn_01x03, J5 Conn_01x03, J9 Conn_01x06, SW1 SW_SPDT, U2 STM32G474RETx, U3 AZ1117-3.3

Commit message: update pcb
Routing:
- net SPI_RST: track 37.5 -> 35.7 mm
- net SPI_DC: track 36.4 -> 34.8 mm
- net NRST: track 30.0 -> 30.5 mm
Changed lines of the file:
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@@
 			(drillshape 0)
 			(scaleselection 1)
-			(outputdirectory "./")
+			(outputdirectory "gerbers/")
 		)
 	)
@@
 	)
 	(segment
-		(start 154.55 101.45)
-		(end 159.4 106.3)
+		(start 167.05 117.65)
+		(end 168.55 117.65)
 		(width 0.2)
 		(layer "F.Cu")
@@
 	)
 	(segment
-		(start 166.6 117.2)
-		(end 167.05 117.65)
+		(start 154.55 101.45)
+		(end 159.4 106.3)
 		(width 0.2)
 		(layer "F.Cu")
@@
 	)
 	(segment
-		(start 167.05 117.65)
-		(end 168.55 117.65)
+		(start 165.5 117)
+		(end 166.4 117)
 		(width 0.2)
 		(layer "F.Cu")
@@
 	)
 	(segment
+		(start 166.4 117)
+		(end 167.05 117.65)
+		(width 0.2)
+		(layer "F.Cu")
+		(net 4)
+	)
+	(segment
 		(start 149.525 101.45)
 		(end 154.55 101.45)
@@
 	)
 	(via
-		(at 166.6 117.2)
+		(at 165.5 117)
 		(size 0.45)
 		(drill 0.3)
@@
 	)
 	(segment
-		(start 166.6 113.5)
-		(end 166.6 117.2)
+		(start 165.5 117)
+		(end 165.5 112.4)
 		(width 0.2)
 		(layer "B.Cu")
@@
 	)
 	(segment
-		(start 159.4 106.3)
-		(end 166.6 113.5)
+		(start 165.5 112.4)
+		(end 159.4 106.3)
 		(width 0.2)
 		(layer "B.Cu")
@@
 	(segment
 		(start 147.575 113.61759)
-		(end 147.575 116.175)
+		(end 147.575 114.425)
 		(width 0.2)
 		(layer "F.Cu")
@@
 	)
 	(segment
-		(start 147.575 116.175)
-		(end 149.2 117.8)
+		(start 150.8 118.575)
+		(end 149.975 118.575)
 		(width 0.2)
 		(layer "F.Cu")
@@
 	)
 	(segment
-		(start 147.575 114.425)
+		(start 147.575 116.175)
 		(end 147.575 113.61759)
 		(width 0.2)
@@
 		(net 25)
 	)
+	(segment
+		(start 149.975 118.575)
+		(end 147.575 116.175)
+		(width 0.2)
+		(layer "F.Cu")
+		(net 25)
+	)
 	(via
-		(at 149.2 117.8)
+		(at 150.8 118.575)
 		(size 0.45)
 		(drill 0.3)
@@
 	)
 	(segment
-		(start 149.2 117.8)
-		(end 149.7 118.3)
+		(start 150.8 118.575)
+		(end 151.075 118.3)
 		(width 0.2)
 		(layer "B.Cu")
@@
 	)
 	(segment
-		(start 166.4 118.3)
-		(end 170.8 113.9)
+		(start 151.075 118.3)
+		(end 166.4 118.3)
 		(width 0.2)
 		(layer "B.Cu")
@@
 	)
 	(segment
-		(start 170.8 108.7)
-		(end 173.5 106)
+		(start 170.8 113.9)
+		(end 170.8 108.7)
 		(width 0.2)
 		(layer "B.Cu")
@@
 	)
 	(segment
-		(start 149.7 118.3)
-		(end 166.4 118.3)
+		(start 166.4 118.3)
+		(end 170.8 113.9)
 		(width 0.2)
 		(layer "B.Cu")
@@
 	)
 	(segment
-		(start 170.8 113.9)
-		(end 170.8 108.7)
+		(start 170.8 108.7)
+		(end 173.5 106)
 		(width 0.2)
 		(layer "B.Cu")
@@
 	)
 	(segment
-		(start 146.575 116.675)
+		(start 146.575 116.375)
 		(end 146.575 114.425)
 		(width 0.2)
@@
 	)
 	(segment
-		(start 149.8 119.9)
-		(end 146.575 116.675)
+		(start 150.1 119.9)
+		(end 146.575 116.375)
 		(width 0.2)
 		(layer "F.Cu")
@@
 	(segment
 		(start 151.6 119.9)
-		(end 149.8 119.9)
+		(end 150.1 119.9)
 		(width 0.2)
 		(layer "F.Cu")
@@
 	)
 	(segment
-		(start 168.1 120)
-		(end 173.5 114.6)
+		(start 152.398 119.102)
+		(end 166.7322 119.102)
 		(width 0.2)
 		(layer "B.Cu")
@@
 	)
 	(segment
-		(start 151.7 120)
-		(end 168.1 120)
+		(start 173.5 112.3342)
+		(end 173.5 111)
 		(width 0.2)
 		(layer "B.Cu")
@@
 	(segment
 		(start 151.6 119.9)
-		(end 151.7 120)
+		(end 152.398 119.102)
 		(width 0.2)
 		(layer "B.Cu")
@@
 	)
 	(segment
-		(start 173.5 114.6)
-		(end 173.5 111)
+		(start 166.7322 119.102)
+		(end 173.5 112.3342)
 		(width 0.2)
 		(layer "B.Cu")
@@
 	(segment
 		(start 151.5 119.1)
-		(end 149.565686 119.1)
+		(end 149.9 119.1)
 		(width 0.2)
 		(layer "F.Cu")
@@
 	)
 	(segment
-		(start 147.075 116.609314)
+		(start 147.075 116.275)
 		(end 147.075 114.425)
 		(width 0.2)
@@
 	)
 	(segment
-		(start 149.565686 119.1)
-		(end 147.075 116.609314)
+		(start 149.9 119.1)
+		(end 147.075 116.275)
 		(width 0.2)
 		(layer "F.Cu")
@@
 	)
 	(segment
-		(start 171.2 116.334314)
-		(end 171.2 110.8)
+		(start 166.199 118.701)
+		(end 166.2339 118.701)
 		(width 0.2)
 		(layer "B.Cu")
@@
 	)
 	(segment
-		(start 171.2 110.8)
-		(end 173.5 108.5)
+		(start 166.5661 118.701)
+		(end 166.801 118.4661)
 		(width 0.2)
 		(layer "B.Cu")
@@
 	)
 	(segment
-		(start 168.134314 119.4)
-		(end 171.2 116.334314)
+		(start 171.201 113.7339)
+		(end 171.201 110.799)
 		(width 0.2)
 		(layer "B.Cu")
@@
 	(segment
 		(start 151.648529 119.1)
-		(end 151.948529 119.4)
+		(end 152.047529 118.701)
 		(width 0.2)
 		(layer "B.Cu")
@@
 	)
 	(segment
-		(start 151.948529 119.4)
-		(end 168.134314 119.4)
+		(start 170.9661 114.301)
+		(end 171.201 114.0661)
+		(width 0.2)
+		(layer "B.Cu")
+		(net 27)
+	)
+	(segment
+		(start 152.047529 118.701)
+		(end 166.199 118.701)
+		(width 0.2)
+		(layer "B.Cu")
+		(net 27)
+	)
+	(segment
+		(start 171.201 110.799)
+		(end 173.5 108.5)
+		(width 0.2)
+		(layer "B.Cu")
+		(net 27)
+	)
+	(segment
+		(start 166.2339 118.701)
+		(end 166.5661 118.701)
+		(width 0.2)
+		(layer "B.Cu")
+		(net 27)
+	)
+	(segment
+		(start 166.801 118.4661)
+		(end 170.9661 114.301)
+		(width 0.2)
+		(layer "B.Cu")
+		(net 27)
+	)
+	(segment
+		(start 171.201 114.0661)
+		(end 171.201 113.7339)
 		(width 0.2)
 		(layer "B.Cu")
@@
 		(hatch edge 0.5)
 		(connect_pads
-			(clearance 0.2)
+			(clearance 0.3)
 		)
 		(min_thickness 0.25)
